File: keyboard/keyboard.kicad_pcb (KiCad board)
At the start: 2 copper layers, 10 x 10 mm, 137 parts, among them J1 SW_SPST, K1 SW_SPST, M1 SW_SPST, P1 SW_SPST, Q1 SW_SPST, SW1 S', T1 SW_SPST, U1 Teensy2.0_(C), U2 SW_SPST, X1 SW_SPST, Y1 SW_SPST

Commit message: Worked on PCB Layout
Parts:
- Alt2, Ctrl2: footprint Button_Switch_Keyboard:SW_Cherry_MX_1.25u_Plate -> Button_Switch_Keyboard:SW_Cherry_MX_1.00u_Plate
- D1, D10, D11, D12, D13, D14, D15, D16, D17, D18, D2, D20, D21, D22, D23, D24, D25, D26, D27, D28, D29, D3, D30, D31, D32, D33, D34, D35, D36, D37, D38, D39, D4, D40, D41, D42, D43, D44, D45, D46, D47, D48, D49, D5, D50, D51, D52, D53, D54, D55, D56, D57, D58, D59, D6, D60, D61, D62, D63, D64, D66, D67, D68, D69, D7, D8, D9: moved to B.Cu
- S`1: renamed from SW1; value S' -> SW_SPST
- moved D67 586.4 mm to (294.0, -38.1), turned to 90 degrees
- moved D65 583.9 mm to (298.6, -80.0), turned to 90 degrees
- moved D66 582.9 mm to (298.6, -61.0), turned to 90 degrees
- moved D52 579.8 mm to (232.0, -61.0), turned to 90 degrees
- moved D68 568.4 mm to (292.7, -20.4), turned to 90 degrees
- moved D60 560.9 mm to (270.1, -80.0), turned to 90 degrees
- moved Enter1 553.6 mm to (264.8, -50.6)
- moved S\1 551.7 mm to (271.9, -69.7)
- moved D57 548.4 mm to (251.0, -61.0), turned to 90 degrees
- moved D69 547.2 mm to (293.8, -1.60), turned to 90 degrees
- moved D61 546.6 mm to (274.8, -61.0), turned to 90 degrees
- moved D42 546.2 mm to (193.9, -61.0), turned to 90 degrees
- moved D59 542.1 mm to (254.9, -1.90), turned to 90 degrees
- moved D62 541.7 mm to (262.2, -37.6), turned to 90 degrees
- moved D41 540.8 mm to (184.3, -80.0), turned to 90 degrees
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- renumbered I1 to I17
Other:
- board size 10 x 10 mm -> 302.5 x 93 mm

Commit message: Continued work on wiring
Parts:
- D65: moved to B.Cu
- moved U1 219.1 mm to (16.6, -104.7)
- moved D58 6.95 mm to (253.4, -22.9)
- moved D62 6.94 mm to (267.7, -41.9)
- moved D3 6.84 mm to (20.0, -41.9)
- moved D63 6.70 mm to (279.6, -22.9)
- moved D14 6.64 mm to (62.9, -3.80)
- moved D13 6.55 mm to (55.8, -22.9)
- moved D23 6.53 mm to (93.9, -22.9)
- moved D18 6.51 mm to (74.8, -22.9)
- moved D68 6.42 mm to (298.6, -22.9)
- moved D48 6.26 mm to (217.7, -41.9)
- moved D2 6.16 mm to (241.5, -3.80)
- moved D8 6.15 mm to (46.2, -41.9)
- moved D17 6.14 mm to (84.3, -41.9)
- moved D27 6.14 mm to (112.9, -22.9)
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- renumbered D55 to D2
Routing:
- net Net-(Delete1-Pad2): track 0.00 -> 438.0 mm
- net Net-(Backspace1-Pad2): track 0.00 -> 425.2 mm
- net Net-(Left1-Pad2): track 0.00 -> 399.6 mm
- net Net-(D14-Pad1): track 0.00 -> 399.2 mm
- net Net-(Ctrl2-Pad2): track 0.00 -> 385.3 mm
- net Net-(D13-Pad1): track 0.00 -> 354.6 mm
- net Net-(D12-Pad1): track 0.00 -> 339.2 mm
- net Net-(D11-Pad1): track 0.00 -> 322.9 mm
- net Net-(D1-Pad1): track 0.00 -> 307.7 mm
- net Net-(Caps_Lock1-Pad2): track 0.00 -> 117.5 mm
- net Net-(Fn1-Pad2): track 0.00 -> 92.2 mm
- net Net-(Alt2-Pad2): track 0.00 -> 92.0 mm
- net Net-(Alt1-Pad2): track 0.00 -> 89.5 mm
- net Net-(B1-Pad2): track 0.00 -> 87.1 mm
- net Net-(A1-Pad2): track 0.00 -> 85.2 mm
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Other:
- board size 302.5 x 93 mm -> 302.5 x 116 mm
